Commit message: Updated urdf for camera and lidar

File: model_pkg/model/ardc_urdf.xacro (robot description, xacro)
@@ -18,4 +18,11 @@
   <xacro:property name="castor_wheel_radius" value="0.035"/>
   <xacro:property name="castor_wheel_width" value="0.01867"/>
+  <xacro:property name="M_PI" value="3.1415926535897931" />
+  <xacro:property name="laser_min_range" value="0.1"/>
+  <xacro:property name="laser_max_range" value="200.0"/>
+  <xacro:property name="samples" value="40000"/>
+  <xacro:property name="resolution" value="0.002"/>
+  <xacro:property name="noise_mean" value="0.0"/>
+  <xacro:property name="noise_stddev" value="0.01"/>
   <xacro:property name="M_PI" value="3.1415926535897931"/>
   <!-- ============================= -->
@@ -70,6 +77,6 @@
     <parent link="base_link"/>
     <child link="left_wheel"/>
-    <origin xyz="${wheel_x_offset} ${wheel_y_offset} 0" rpy="0 0 1.57"/>
-    <axis xyz="0 1 0"/>
+    <origin xyz="${wheel_x_offset} -${wheel_y_offset} 0" rpy="0 0 1.57"/>
+    <axis xyz="-1 0 0"/>
   </joint>
   <gazebo reference="left_wheel">
@@ -98,6 +105,6 @@
     <parent link="base_link"/>
     <child link="right_wheel"/>
-    <origin xyz="${wheel_x_offset} -${wheel_y_offset} 0" rpy="0 0 1.57"/>
-    <axis xyz="0 1 0"/>
+    <origin xyz="${wheel_x_offset} ${wheel_y_offset} 0" rpy="0 0 1.57"/>
+    <axis xyz="-1 0 0"/>
   </joint>
   <gazebo reference="right_wheel">
@@ -123,5 +130,5 @@
     </inertial>
   </link>
-  <joint name="connecting_rod_joint" type="continuous">
+  <joint name="connecting_rod_joint" type="fixed">
     <parent link="base_link"/>
     <child link="connecting_rod"/>
@@ -137,10 +144,10 @@
   <link name="castor_wheel">
     <visual>
-      <geometry><cylinder length="${castor_wheel_width}" radius="${castor_wheel_radius}"/></geometry>
+      <geometry><sphere radius="${castor_wheel_radius}"/></geometry>
       <origin xyz="0 0 0" rpy="0 1.5708 0"/>
       <material name="black_rubber"/>
     </visual>
     <collision>
-      <geometry><cylinder length="${castor_wheel_width}" radius="${castor_wheel_radius}"/></geometry>
+      <geometry><sphere radius="${castor_wheel_radius}"/></geometry>
       <origin xyz="0 0 0" rpy="0 1.5708 0"/>
     </collision>
@@ -151,5 +158,5 @@
     </inertial>
   </link>
-  <joint name="castor_wheel_joint" type="continuous">
+  <joint name="castor_wheel_joint" type="fixed">
     <parent link="connecting_rod"/>
     <child link="castor_wheel"/>
@@ -164,7 +171,7 @@
   <!-- ============================= -->
   <link name="base_footprint"/>
-  <joint name="base_joint" type="fixed">
-    <parent link="base_footprint"/>
-    <child link="base_link"/>
+  <joint name="base_footprint_joint" type="fixed">
+    <parent link="base_link"/>
+    <child link="base_footprint"/>
     <origin xyz="0 0 0" rpy="0 0 0"/>
   </joint>
@@ -194,3 +201,135 @@
   </plugin>
   </gazebo>
+  <!-- ============================= -->
+  <!-- LIDAR -->
+  <!-- ============================= -->
+  <link name="lidar_link">
+    <visual>
+      <geometry>
+        <box size="0.1 0.1 0.1"/>
+      </geometry>
+      <origin rpy="0 0 0" xyz="0 0 0"/>
+    </visual>
+    <collision>
+      <geometry>
+        <box size="0.1 0.1 0.1"/>
+      </geometry>
+      <origin rpy="0 0 0" xyz="0 0 0"/>
+    </collision>
+    <inertial>
+      <mass value="0.05"/>
+      <origin rpy="0 0 0" xyz="0 0 0"/>
+      <inertia ixx="0.001" ixy="0" ixz="0" iyy="0.001" iyz="0" izz="0.001"/>
+    </inertial>
+  </link>
+  <joint name="lidar_joint" type="fixed">
+    <parent link="base_link"/>
+    <child link="lidar_link"/>
+    <origin xyz="-0.32 0 0.4" rpy="0 0 0"/>
+  </joint>
+  <gazebo reference="lidar_link">
+    <sensor type="gpu_ray" name="lidar-VLP16">
+      <pose>0 0 0 0 0 0</pose>
+      <visualize>false</visualize>
+      <update_rate>40</update_rate>
+      <ray>
+        <scan>
+          <horizontal>
+          <samples>100</samples>
+          <resolution>1</resolution>
+          <min_angle>${0}</min_angle>
+          <max_angle>${2*M_PI}</max_angle>
+          </horizontal>
+          <vertical>
+          <samples>360</samples>
+          <resolution>1</resolution>
+          <min_angle>${-7.22/180*M_PI}</min_angle>
+          <max_angle>${55.22/180*M_PI}</max_angle>
+          </vertical>
+          </scan>
+          <range>
+          <min>${laser_min_range}</min>
+          <max>${laser_max_range}</max>
+          <resolution>${resolution}</resolution>
+          </range>
+          <noise>
+          <type>gaussian</type>
+          <mean>${noise_mean}</mean>
+          <stddev>${noise_stddev}</stddev>
+          </noise>
+      </ray>
+      <plugin name="gazebo_ros_laser_controller" filename="libgazebo_ros_ray_sensor.so">
+      <outputType>sensor_msgs/PointCloud2</outputType>
+      <topicName>Lidar/PointCloud</topicName>
+      <frameName>lidar_link</frameName>
+      </plugin>
+    </sensor>
+  </gazebo>
+  <!-- ============================= -->
+  <!-- Camera -->
+  <!-- ============================= -->
+  <link name="camera_link">
+    <collision>
+      <origin xyz="0 0 0" rpy="0 0 0"/>
+      <geometry>
+    <box size="0.1 0.1 0.1"/>
+      </geometry>
+    </collision>
+    <visual>
+      <origin xyz="0 0 0" rpy="0 0 0"/>
+      <geometry>
+    <box size="0.1 0.1 0.1"/>
+      </geometry>
+      <material name="red"/>
+    </visual>
+    <inertial>
+      <mass value="1e-5" />
+      <origin xyz="0 0 0" rpy="0 0 0"/>
+      <inertia ixx="1e-6" ixy="0" ixz="0" iyy="1e-6" iyz="0" izz="1e-6" />
+    </inertial>
+  </link>
+  <joint name="camera_joint" type="fixed">
+    <parent link = "base_link"/>
+    <child link="camera_link"/>
+    <origin xyz="-${base_length/2} 0 ${wheel_radius + base_height}" rpy="0 0.2 3.14"/>
+  </joint>
+  <gazebo reference="camera_link">
+    <sensor type="camera" name="camera_link">
+      <update_rate>30.0</update_rate>
+      <camera name="camera">
+        <horizontal_fov>1.3962634</horizontal_fov>
+        <image>
+          <width>1600</width>
+          <height>900</height>
+          <format>R8G8B8</format>
+        </image>
+        <clip>
+          <near>0.02</near>
+          <far>300</far>
+        </clip>
+        <noise>
+          <type>gaussian</type>
+          <!-- Noise is sampled independently per pixel on each frame.
+               That pixel's noise value is added to each of its color
+               channels, which at that point lie in the range [0,1]. -->
+          <mean>0.0</mean>
+          <stddev>0.007</stddev>
+        </noise>
+      </camera>
+      <plugin name="camera_controller" filename="libgazebo_ros_camera.so">
+        <alwaysOn>true</alwaysOn>
+        <updateRate>0.0</updateRate>
+        <camera_name>camera</camera_name>
+        <imageTopicName>image_raw</imageTopicName>
+        <cameraInfoTopicName>camera_info</cameraInfoTopicName>
+        <frameName>camera_link</frameName>
+        <hackBaseline>0.07</hackBaseline>
+        <distortionK1>0.0</distortionK1>
+        <distortionK2>0.0</distortionK2>
+        <distortionK3>0.0</distortionK3>
+        <distortionT1>0.0</distortionT1>
+        <distortionT2>0.0</distortionT2>
+      </plugin>
+    </sensor>
+  </gazebo>
 </robot>

Commit message: Added IMU and GPS in the urdf

File: model_pkg/model/ardc_urdf.xacro (robot description, xacro)
@@ -336,3 +336,152 @@
     </sensor>
   </gazebo>
+<!-- ============================= -->
+<!-- IMU -->
+<!-- ============================= -->
+<link name="imu_link">
+  <visual>
+    <geometry>
+      <box size="0.1 0.1 0.1"/>
+    </geometry>
+  </visual>
+  <collision>
+    <geometry>
+      <box size="0.1 0.1 0.1"/>
+    </geometry>
+  </collision>
+  <inertial>
+    <mass value="0.01"/>
+    <inertia ixx="0.001" ixy="0" ixz="0" iyy="0.001" iyz="0" izz="0.001"/>
+  </inertial>
+</link>
+<joint name="imu_joint" type="fixed">
+  <parent link="base_link"/>
+  <child link="imu_link"/>
+  <origin xyz="0 0 0.01"/>
+</joint>
+<gazebo reference="imu_link">
+  <sensor name="imu_sensor" type="imu">
+   <plugin filename="libgazebo_ros_imu_sensor.so" name="imu_plugin">
+      <ros>
+        <remapping>~/out:=/imu/data</remapping>
+      </ros>
+      <initial_orientation_as_reference>false</initial_orientation_as_reference>
+    </plugin>
+    <always_on>true</always_on>
+    <update_rate>100</update_rate>
+    <visualize>true</visualize>
+    <imu>
+      <angular_velocity>
+        <x>
+          <noise type="gaussian">
+            <mean>0.0</mean>
+            <stddev>2e-4</stddev>
+            <bias_mean>0.0000075</bias_mean>
+            <bias_stddev>0.0000008</bias_stddev>
+          </noise>
+        </x>
+        <y>
+          <noise type="gaussian">
+            <mean>0.0</mean>
+            <stddev>2e-4</stddev>
+            <bias_mean>0.0000075</bias_mean>
+            <bias_stddev>0.0000008</bias_stddev>
+          </noise>
+        </y>
+        <z>
+          <noise type="gaussian">
+            <mean>0.0</mean>
+            <stddev>2e-4</stddev>
+            <bias_mean>0.0000075</bias_mean>
+            <bias_stddev>0.0000008</bias_stddev>
+          </noise>
+        </z>
+      </angular_velocity>
+      <linear_acceleration>
+        <x>
+          <noise type="gaussian">
+            <mean>0.0</mean>
+            <stddev>1.7e-2</stddev>
+            <bias_mean>0.1</bias_mean>
+            <bias_stddev>0.001</bias_stddev>
+          </noise>
+        </x>
+        <y>
+          <noise type="gaussian">
+            <mean>0.0</mean>
+            <stddev>1.7e-2</stddev>
+            <bias_mean>0.1</bias_mean>
+            <bias_stddev>0.001</bias_stddev>
+          </noise>
+        </y>
+        <z>
+          <noise type="gaussian">
+            <mean>0.0</mean>
+            <stddev>1.7e-2</stddev>
+            <bias_mean>0.1</bias_mean>
+            <bias_stddev>0.001</bias_stddev>
+          </noise>
+        </z>
+      </linear_acceleration>
+    </imu>
+  </sensor>
+</gazebo>
+<!-- ============================= -->
+<!-- GPS -->
+<!-- ============================= -->
+<link name="gps_link">
+  <collision>
+    <origin xyz="0 0 0" rpy="0 0 0"/>
+    <geometry>
+    <box size="0.1 0.1 0.1"/>
+    </geometry>
+  </collision>
+  <visual>
+    <origin xyz="0 0 0" rpy="0 0 0"/>
+    <geometry>
+    <box size="0.1 0.1 0.1"/>
+    </geometry>
+  </visual>
+  <inertial>
+    <mass value="1e-5" />
+    <origin xyz="0 0 0" rpy="0 0 0"/>
+    <inertia ixx="1e-6" ixy="0" ixz="0" iyy="1e-6" iyz="0" izz="1e-6" />
+  </inertial>
+</link>
+<joint name="gps_joint" type="fixed">
+  <parent link="base_link"/>
+  <child link="gps_link"/>
+  <origin xyz="0 0 0" rpy="0 0 0"/>
+</joint>
+ <gazebo reference="gps_link">
+	<sensor name="bot_gps" type="gps">
+	  <always_on>true</always_on>
+	  <update_rate>1</update_rate>
+	  <pose>0 0 0 0 0 0</pose>
+	  <gps>
+	    <position_sensing>
+	      <horizontal>
+		<noise type="gaussian">
+		  <mean>0.0</mean>
+		  <stddev>0.01</stddev>
+		</noise>
+	      </horizontal>
+	      <vertical>
+		<noise type="gaussian">
+		  <mean>0.0</mean>
+		  <stddev>0.01</stddev>
+		</noise>
+	      </vertical>
+	    </position_sensing>
+	  </gps>
+	  <plugin name="my_gps_plugin" filename="libgazebo_ros_gps_sensor.so">
+	    <ros>
+	      <namespace>gps</namespace>
+	      <remapping>~/out:=/gpsfix</remapping>
+	    </ros>
+	    <output_type>sensor_msgs/NavSatFix</output_type>
+            <frame_name>gps_link</frame_name>
+	  </plugin>
+	</sensor>
+   </gazebo>
 </robot>

Commit message: updated urdf and liv=dar processing config

File: model_pkg/model/ardc_urdf.xacro (robot description, xacro)
@@ -24,5 +24,5 @@
   <xacro:property name="resolution" value="0.002"/>
   <xacro:property name="noise_mean" value="0.0"/>
-  <xacro:property name="noise_stddev" value="0.01"/>
+  <xacro:property name="noise_stddev" value="0.0"/>
   <xacro:property name="M_PI" value="3.1415926535897931"/>
   <!-- ============================= -->
@@ -194,6 +194,6 @@
     <max_wheel_acceleration>1.0</max_wheel_acceleration>
     <!-- output -->
-    <publish_odom>true</publish_odom>
-    <publish_odom_tf>true</publish_odom_tf>
+    <publish_odom>false</publish_odom>        <!-- odom topic -->
+    <publish_odom_tf>true</publish_odom_tf>   <!-- odom frame -->
     <publish_wheel_tf>true</publish_wheel_tf>
     <odometry_frame>odom</odometry_frame>
@@ -226,5 +226,5 @@
     <parent link="base_link"/>
     <child link="lidar_link"/>
-    <origin xyz="-0.32 0 0.4" rpy="0 0 0"/>
+    <origin xyz="0.0 0 0.6" rpy="0 0 0"/>
   </joint>
   <gazebo reference="lidar_link">
@@ -361,8 +361,8 @@
   <origin xyz="0 0 0.01"/>
 </joint>
-<gazebo reference="imu_link">
+<gazebo reference="lidar_link">
   <sensor name="imu_sensor" type="imu">
    <plugin filename="libgazebo_ros_imu_sensor.so" name="imu_plugin">
-   <frameName>imu_link</frameName>
+   <frameName>lidar_link</frameName>
       <ros>
         <remapping>~/out:=/imu/data</remapping>
@@ -371,5 +371,5 @@
     </plugin>
     <always_on>true</always_on>
-    <update_rate>100</update_rate>
+    <update_rate>500</update_rate>
     <visualize>true</visualize>
     <imu>
@@ -378,7 +378,7 @@
           <noise type="gaussian">
             <mean>0.0</mean>
-            <stddev>2e-4</stddev>
-            <bias_mean>0.0000075</bias_mean>
-            <bias_stddev>0.0000008</bias_stddev>
+            <stddev>0.0</stddev>
+            <bias_mean>0.0</bias_mean>
+            <bias_stddev>0.0</bias_stddev>
           </noise>
         </x>
@@ -386,7 +386,7 @@
           <noise type="gaussian">
             <mean>0.0</mean>
-            <stddev>2e-4</stddev>
-            <bias_mean>0.0000075</bias_mean>
-            <bias_stddev>0.0000008</bias_stddev>
+            <stddev>0.0</stddev>
+            <bias_mean>0.0</bias_mean>
+            <bias_stddev>0.0</bias_stddev>
           </noise>
         </y>
@@ -394,7 +394,7 @@
           <noise type="gaussian">
             <mean>0.0</mean>
-            <stddev>2e-4</stddev>
-            <bias_mean>0.0000075</bias_mean>
-            <bias_stddev>0.0000008</bias_stddev>
+            <stddev>0.0</stddev>
+            <bias_mean>0.0</bias_mean>
+            <bias_stddev>0.0</bias_stddev>
           </noise>
         </z>
@@ -404,7 +404,7 @@
           <noise type="gaussian">
             <mean>0.0</mean>
-            <stddev>1.7e-2</stddev>
-            <bias_mean>0.1</bias_mean>
-            <bias_stddev>0.001</bias_stddev>
+            <stddev>0.0</stddev>
+            <bias_mean>0.0</bias_mean>
+            <bias_stddev>0.0</bias_stddev>
           </noise>
         </x>
@@ -412,7 +412,7 @@
           <noise type="gaussian">
             <mean>0.0</mean>
-            <stddev>1.7e-2</stddev>
-            <bias_mean>0.1</bias_mean>
-            <bias_stddev>0.001</bias_stddev>
+            <stddev>0.0</stddev>
+            <bias_mean>0.0</bias_mean>
+            <bias_stddev>0.0</bias_stddev>
           </noise>
         </y>
@@ -420,7 +420,7 @@
           <noise type="gaussian">
             <mean>0.0</mean>
-            <stddev>1.7e-2</stddev>
-            <bias_mean>0.1</bias_mean>
-            <bias_stddev>0.001</bias_stddev>
+            <stddev>0.0</stddev>
+            <bias_mean>0.0</bias_mean>
+            <bias_stddev>0.0</bias_stddev>
           </noise>
         </z>

Commit message: added navigation packages

File: model_pkg/model/ardc_urdf.xacro (robot description, xacro)
@@ -26,4 +26,5 @@
   <xacro:property name="noise_stddev" value="0.0"/>
   <xacro:property name="M_PI" value="3.1415926535897931"/>
+  <xacro:include filename="$(find ros2_livox_simulation)/urdf/mid360.xacro" />
   <!-- ============================= -->
   <!-- MATERIALS (for RViz) -->
@@ -172,7 +173,7 @@
   <link name="base_footprint"/>
   <joint name="base_footprint_joint" type="fixed">
-    <parent link="base_link"/>
-    <child link="base_footprint"/>
-    <origin xyz="0 0 0" rpy="0 0 0"/>
+    <parent link="base_footprint"/>
+    <child link="base_link"/>
+    <origin xyz="0 0 0" rpy="0 0 ${M_PI}"/>
   </joint>
   <!-- ============================= -->
@@ -194,9 +195,9 @@
     <max_wheel_acceleration>1.0</max_wheel_acceleration>
     <!-- output -->
-    <publish_odom>false</publish_odom>        <!-- odom topic -->
-    <publish_odom_tf>true</publish_odom_tf>   <!-- odom frame -->
+    <publish_odom>true</publish_odom>        <!-- odom topic -->
+    <publish_odom_tf>false</publish_odom_tf>   <!-- odom frame -->
     <publish_wheel_tf>true</publish_wheel_tf>
     <odometry_frame>odom</odometry_frame>
-    <robot_base_frame>base_link</robot_base_frame>
+    <robot_base_frame>base_footprint</robot_base_frame>
   </plugin>
   </gazebo>
@@ -205,5 +206,5 @@
   <!-- ============================= -->
   <link name="lidar_link">
-    <visual>
+    <!-- <visual>
       <geometry>
         <box size="0.1 0.1 0.1"/>
@@ -221,5 +222,5 @@
       <origin rpy="0 0 0" xyz="0 0 0"/>
       <inertia ixx="0.001" ixy="0" ixz="0" iyy="0.001" iyz="0" izz="0.001"/>
-    </inertial>
+    </inertial> -->
   </link>
   <joint name="lidar_joint" type="fixed">
@@ -228,5 +229,5 @@
     <origin xyz="0.0 0 0.6" rpy="0 0 0"/>
   </joint>
-  <gazebo reference="lidar_link">
+  <!-- <gazebo reference="lidar_link">
     <sensor type="gpu_ray" name="lidar-Livox-mid360">
       <pose>0 0 0 0 0 0</pose>
@@ -264,10 +265,12 @@
         <namespace>/</namespace>
         <remapping>~/out:=/Livox/PointCloud</remapping>
-        <!-- <parameter name="frame_name">lidar_link</parameter>
-        <parameter name="output_type">sensor_msgs/PointCloud2</parameter> -->
       </ros>
       </plugin>
     </sensor>
-  </gazebo>
+  </gazebo> -->
+  <xacro:mid360 name="livox" parent="base_link" topic="livox">
+    <origin xyz="-${base_length/2} 0 ${wheel_radius + base_height}" rpy="0 0 3.14"/>
+    0 ${M_PI/3} 3.14
+  </xacro:mid360>
   <!-- ============================= -->
   <!-- Camera -->
@@ -276,7 +279,7 @@
     <collision>
       <origin xyz="0 0 0" rpy="0 0 0"/>
-      <geometry>
+      <!-- <geometry>
     <box size="0.1 0.1 0.1"/>
-      </geometry>
+      </geometry> -->
     </collision>
     <visual>
@@ -314,7 +317,4 @@
         <noise>
           <type>gaussian</type>
-          <!-- Noise is sampled independently per pixel on each frame.
-               That pixel's noise value is added to each of its color
-               channels, which at that point lie in the range [0,1]. -->
           <mean>0.0</mean>
           <stddev>0.007</stddev>
@@ -361,8 +361,8 @@
   <origin xyz="0 0 0.01"/>
 </joint>
-<gazebo reference="lidar_link">
+<gazebo reference="imu_link">
   <sensor name="imu_sensor" type="imu">
    <plugin filename="libgazebo_ros_imu_sensor.so" name="imu_plugin">
-   <frameName>lidar_link</frameName>
+   <frameName>imu_link</frameName>
       <ros>
         <remapping>~/out:=/imu/data</remapping>
@@ -378,5 +378,5 @@
           <noise type="gaussian">
             <mean>0.0</mean>
-            <stddev>0.0</stddev>
+            <stddev>0.01</stddev>
             <bias_mean>0.0</bias_mean>
             <bias_stddev>0.0</bias_stddev>
@@ -386,5 +386,5 @@
           <noise type="gaussian">
             <mean>0.0</mean>
-            <stddev>0.0</stddev>
+            <stddev>0.01</stddev>
             <bias_mean>0.0</bias_mean>
             <bias_stddev>0.0</bias_stddev>
@@ -394,5 +394,5 @@
           <noise type="gaussian">
             <mean>0.0</mean>
-            <stddev>0.0</stddev>
+            <stddev>0.01</stddev>
             <bias_mean>0.0</bias_mean>
             <bias_stddev>0.0</bias_stddev>
@@ -412,5 +412,5 @@
           <noise type="gaussian">
             <mean>0.0</mean>
-            <stddev>0.0</stddev>
+            <stddev>0.01</stddev>
             <bias_mean>0.0</bias_mean>
             <bias_stddev>0.0</bias_stddev>
@@ -420,5 +420,5 @@
           <noise type="gaussian">
             <mean>0.0</mean>
-            <stddev>0.0</stddev>
+            <stddev>0.01</stddev>
             <bias_mean>0.0</bias_mean>
             <bias_stddev>0.0</bias_stddev>
@@ -466,5 +466,5 @@
 		<noise type="gaussian">
 		  <mean>0.0</mean>
-		  <stddev>0.01</stddev>
+		  <stddev>0.00</stddev>
 		</noise>
 	      </horizontal>
