Commit message: fixed the turning problem

File: model_pkg/model/ardc_urdf.xacro (robot description, xacro)
@@ -78,6 +78,6 @@
     <parent link="base_link"/>
     <child link="left_wheel"/>
-    <origin xyz="${wheel_x_offset} -${wheel_y_offset} 0" rpy="0 0 1.57"/>
-    <axis xyz="-1 0 0"/>
+    <origin xyz="-${wheel_x_offset} -${wheel_y_offset} 0" rpy="0 0 1.57"/>
+    <axis xyz="1 0 0"/>
   </joint>
   <gazebo reference="left_wheel">
@@ -106,6 +106,6 @@
     <parent link="base_link"/>
     <child link="right_wheel"/>
-    <origin xyz="${wheel_x_offset} ${wheel_y_offset} 0" rpy="0 0 1.57"/>
-    <axis xyz="-1 0 0"/>
+    <origin xyz="-${wheel_x_offset} ${wheel_y_offset} 0" rpy="0 0 1.57"/>
+    <axis xyz="1 0 0"/>
   </joint>
   <gazebo reference="right_wheel">
@@ -134,5 +134,5 @@
     <parent link="base_link"/>
     <child link="connecting_rod"/>
-    <origin xyz="${connecting_rod_x_offset} 0 -${connecting_rod_length/2-0.05}" rpy="0 0 0"/>
+    <origin xyz="${base_length + connecting_rod_x_offset} 0 -${connecting_rod_length/2-0.05}" rpy="0 0 0"/>
     <axis xyz="0 0 1"/>
   </joint>
@@ -159,5 +159,5 @@
     </inertial>
   </link>
-  <joint name="castor_wheel_joint" type="fixed">
+  <joint name="castor_wheel_joint" type="continuous">
     <parent link="connecting_rod"/>
     <child link="castor_wheel"/>
@@ -171,10 +171,10 @@
   <!-- Base Footprint -->
   <!-- ============================= -->
-  <link name="base_footprint"/>
+  <!-- <link name="base_footprint"/>
   <joint name="base_footprint_joint" type="fixed">
     <parent link="base_footprint"/>
     <child link="base_link"/>
     <origin xyz="0 0 0" rpy="0 0 ${M_PI}"/>
-  </joint>
+  </joint> -->
   <!-- ============================= -->
   <!-- Differential Drive -->
@@ -186,6 +186,6 @@
     </ros>
     <!-- wheels -->
-    <left_joint>left_wheel_joint</left_joint>
-    <right_joint>right_wheel_joint</right_joint>
+    <left_joint>right_wheel_joint</left_joint>
+    <right_joint>left_wheel_joint</right_joint>
     <!-- kinematics -->
     <wheel_separation>${2*wheel_y_offset}</wheel_separation>
@@ -194,10 +194,12 @@
     <max_wheel_torque>20</max_wheel_torque>
     <max_wheel_acceleration>1.0</max_wheel_acceleration>
+    <!-- input -->
+    <command_topic>cmd_vel</command_topic>
     <!-- output -->
     <publish_odom>true</publish_odom>        <!-- odom topic -->
-    <publish_odom_tf>false</publish_odom_tf>   <!-- odom frame -->
+    <publish_odom_tf>true</publish_odom_tf>   <!-- odom frame -->
     <publish_wheel_tf>true</publish_wheel_tf>
     <odometry_frame>odom</odometry_frame>
-    <robot_base_frame>base_footprint</robot_base_frame>
+    <robot_base_frame>base_link</robot_base_frame>
   </plugin>
   </gazebo>

File: model_pkg/model/robot.xacro (robot description, xacro)
@@ -1,29 +1,63 @@
 <?xml version="1.0"?>
-<robot xmlns:xacro="http://www.ros.org/wiki/xacro" name="igvc_robot">
-  <xacro:property name="base_link_length" value="0.5"/>
-  <xacro:property name="base_link_radius" value="0.4"/>
-  <xacro:property name="M_PI" value="3.1415926535897931" />
-  <xacro:property name="laser_min_range" value="0.1"/>
-  <xacro:property name="laser_max_range" value="200.0"/>
-  <xacro:property name="samples" value="40000"/>
-  <xacro:property name="resolution" value="0.002"/>
-  <xacro:property name="noise_mean" value="0.0"/>
-  <xacro:property name="noise_stddev" value="0.01"/>
-  <xacro:property name="mass" value="0.4" />
-  <xacro:property name="length" value="0.1" />
-  <xacro:property name="width" value="0.06" />
-  <xacro:property name="height" value="0.06" />
-  <!-- Dummy Link and Joint -->
-  <link name="base_footprint">
-  </link>
-  <!-- <joint name="dummy_joint" type="fixed">
-    <parent link="base_link"/>
-    <child link="base_link2"/>
-  </joint> -->
-  <!-- Base Link -->
+<robot name="vnymous">
+  <link name="base_footprint"/>
   <link name="base_link">
     <visual>
+      <origin rpy="0 -0 1.5707" xyz="0 0.35 0"/>
       <geometry>
-        <box size="1 0.5 0.1"/>
+        <mesh filename="file://home/abhiyaan-orin/isaac_ros-dev/src/isaac_ros_common/src/vsim/meshes/igvc/igvc_bot.dae" scale="0.001 0.001 0.001"/>
+      </geometry>
+    </visual>
+    <collision>
+      <origin rpy="0 -0 1.5707" xyz="0 0.35 0"/>
+      <geometry>
+        <mesh filename="file://home/abhiyaan-orin/isaac_ros-dev/src/isaac_ros_common/src/vsim/meshes/igvc/igvc_bot.dae" scale="0.001 0.001 0.001"/>
+      </geometry>
+    </collision>
+    <inertial>
+      <mass value="10"/>
+      <inertia ixx="0.166667" ixy="0.0" ixz="0.0" iyy="0.166667" iyz="0.0" izz="0.166667"/>
+    </inertial>
+  </link>
+  <link name="wheel1">
+    <visual>
+      <geometry>
+        <mesh filename="file://home/abhiyaan-orin/isaac_ros-dev/src/isaac_ros_common/src/vsim/meshes/igvc/igvc_wheel.dae" scale="0.001 0.001 0.001"/>
+      </geometry>
+      <origin rpy ="0 0 0" xyz="0 0 0"/>
+    </visual>
+    <collision>
+      <geometry>
+        <cylinder radius="0.12" length="0.04"/>
+      </geometry>
+      <origin rpy ="1.5707 0 1.5707" xyz="-0.065 0 0"/>
+    </collision>
+    <inertial>
+      <mass value="5"/>
+      <inertia ixx="0.166667" ixy="0.0" ixz="0.0" iyy="0.166667" iyz="0.0" izz="0.166667"/>
+    </inertial>
+  </link>
+  <link name="wheel2">
+    <visual>
+      <geometry>
+        <mesh filename="file://home/abhiyaan-orin/isaac_ros-dev/src/isaac_ros_common/src/vsim/meshes/igvc/igvc_wheel.dae" scale="0.001 0.001 0.001"/>
+      </geometry>
+    <origin rpy ="0 0 0" xyz="0 0 0"/>
+    </visual>
+    <collision>
+      <geometry>
+        <cylinder radius="0.12" length="0.04"/>
+      </geometry>
+      <origin rpy ="1.5707 0 1.5707" xyz="-0.065 0 0"/>
+    </collision>
+    <inertial>
+      <mass value="5"/>
+      <inertia ixx="0.166667" ixy="0.0" ixz="0.0" iyy="0.166667" iyz="0.0" izz="0.166667"/>
+    </inertial>
+  </link>
+  <link name="castor_ball">
+    <visual>
+      <geometry>
+        <sphere radius="0.05"/>
       </geometry>
       <origin rpy="0 0 0" xyz="0 0 0"/>
@@ -31,58 +65,17 @@
     <collision>
       <geometry>
-        <box size="1 0.5 0.1"/>
+        <sphere radius="0.05"/>
       </geometry>
       <origin rpy="0 0 0" xyz="0 0 0"/>
     </collision>
     <inertial>
-      <origin rpy="0 0 0" xyz="0 0 0"/>
-      <mass value="1"/>
-      <inertia ixx="0.083" ixy="0" ixz="0" iyy="0.083" iyz="0" izz="0.083"/>
+      <mass value="3"/>
+      <inertia ixx="0.166667" ixy="0.0" ixz="0.0" iyy="0.166667" iyz="0.0" izz="0.166667"/>
     </inertial>
   </link>
-  <!-- Left Wheel Link -->
-  <link name="right_wheel">
+  <link name="castor_cylinder">
     <visual>
       <geometry>
-        <cylinder length="0.1" radius="0.2"/>
-      </geometry>
-      <origin rpy="1.5708 1.5708 0" xyz="0 -0.3 0"/>
-    </visual>
-    <collision>
-      <geometry>
-        <cylinder length="0.1" radius="0.2"/>
-      </geometry>
-      <origin rpy="1.5708 1.5708 0" xyz="0 -0.3 0"/>
-    </collision>
-    <inertial>
-      <origin rpy="1.5708 1.5708 0" xyz="0 -0.3 0"/>
-      <mass value="0.5"/>
-      <inertia ixx="0.006" ixy="0" ixz="0" iyy="0.006" iyz="0" izz="0.001"/>
-    </inertial>
-  </link>
-  <!-- Right Wheel Link -->
-  <link name="left_wheel">
-    <visual>
-      <geometry>
-        <cylinder length="0.1" radius="0.2"/>
-      </geometry>
-      <origin rpy="1.5708 1.5708 0" xyz="0 0.3 0"/>
-    </visual>
-    <collision>
-      <geometry>
-        <cylinder length="0.1" radius="0.2"/>
-      </geometry>
-      <origin rpy="1.5708 1.5708 0" xyz="0 0.3 0"/>
-    </collision>
-    <inertial>
-      <origin rpy="1.5708 1.5708 0" xyz="0 0.3 0"/>
-      <mass value="0.5"/>
-      <inertia ixx="0.006" ixy="0" ixz="0" iyy="0.006" iyz="0" izz="0.001"/>
-    </inertial>
-  </link>
-  <link name="castor_wheel">
-    <visual>
-      <geometry>
-        <sphere radius="0.15"/>
+        <cylinder length="0.03" radius="0.05"/>
       </geometry>
       <origin rpy="0 0 0" xyz="0 0 0"/>
@@ -90,19 +83,17 @@
     <collision>
       <geometry>
-        <sphere radius="0.15"/>
+        <cylinder length="0.03" radius="0.05"/>
       </geometry>
-      <origin rpy="0 0 0" xyz="0 0 0"/>
+      <origin rpy ="0 0 0" xyz="0 0 0"/>
     </collision>
     <inertial>
-      <mass value="0.3"/>
-      <origin rpy="0 0 0" xyz="0 0 0"/>
-      <inertia ixx="0.006" ixy="0" ixz="0" iyy="0.006" iyz="0" izz="0.001"/>
+      <mass value="2"/>
+      <inertia ixx="0.166667" ixy="0.0" ixz="0.0" iyy="0.166667" iyz="0.0" izz="0.166667"/>
     </inertial>
   </link>
-  <!-- Lidar Link -->
-  <link name="lidar_link">
+  <link name="castor_ball2">
     <visual>
       <geometry>
-        <box size="0.1 0.1 0.1"/>
+        <sphere radius="0.05"/>
       </geometry>
       <origin rpy="0 0 0" xyz="0 0 0"/>
@@ -110,99 +101,17 @@
     <collision>
       <geometry>
-        <box size="0.1 0.1 0.1"/>
+        <sphere radius="0.05"/>
       </geometry>
       <origin rpy="0 0 0" xyz="0 0 0"/>
     </collision>
     <inertial>
-      <mass value="0.05"/>
-      <origin rpy="0 0 0" xyz="0 0 0"/>
-      <inertia ixx="0.001" ixy="0" ixz="0" iyy="0.001" iyz="0" izz="0.001"/>
+      <mass value="3"/>
+      <inertia ixx="0.166667" ixy="0.0" ixz="0.0" iyy="0.166667" iyz="0.0" izz="0.166667"/>
     </inertial>
   </link>
-<link name="camera_link_forward">
-    <collision>
-      <origin xyz="0 0 0" rpy="0 0 0"/>
-      <geometry>
-    <box size="0.1 0.1 0.1"/>
-      </geometry>
-    </collision>
-    <visual>
-      <origin xyz="0 0 0" rpy="0 0 0"/>
-      <geometry>
-    <box size="0.1 0.1 0.1"/>
-      </geometry>
-      <material name="red"/>
-    </visual>
-    <inertial>
-      <mass value="1e-5" />
-      <origin xyz="0 0 0" rpy="0 0 0"/>
-      <inertia ixx="1e-6" ixy="0" ixz="0" iyy="1e-6" iyz="0" izz="1e-6" />
-    </inertial>
-  </link>
-<link name="camera_link_backward">
-    <collision>
-      <origin xyz="0 0 0" rpy="0 0 0"/>
-      <geometry>
-    <box size="0.1 0.1 0.1"/>
-      </geometry>
-    </collision>
-    <visual>
-      <origin xyz="0 0 0" rpy="0 0 0"/>
-      <geometry>
-    <box size="0.1 0.1 0.1"/>
-      </geometry>
-      <material name="red"/>
-    </visual>
-    <inertial>
-      <mass value="1e-5" />
-      <origin xyz="0 0 0" rpy="0 0 0"/>
-      <inertia ixx="1e-6" ixy="0" ixz="0" iyy="1e-6" iyz="0" izz="1e-6" />
-    </inertial>
-  </link>
-  <link name="camera_link_left">
-    <collision>
-      <origin xyz="0 0 0" rpy="0 0 0"/>
-      <geometry>
-    <box size="0.1 0.1 0.1"/>
-      </geometry>
-    </collision>
-    <visual>
-      <origin xyz="0 0 0" rpy="0 0 0"/>
-      <geometry>
-    <box size="0.1 0.1 0.1"/>
-      </geometry>
-      <material name="red"/>
-    </visual>
-    <inertial>
-      <mass value="1e-5" />
-      <origin xyz="0 0 0" rpy="0 0 0"/>
-      <inertia ixx="1e-6" ixy="0" ixz="0" iyy="1e-6" iyz="0" izz="1e-6" />
-    </inertial>
-  </link>
-  <link name="camera_link_right">
-    <collision>
-      <origin xyz="0 0 0" rpy="0 0 0"/>
-      <geometry>
-    <box size="0.1 0.1 0.1"/>
-      </geometry>
-    </collision>
-    <visual>
-      <origin xyz="0 0 0" rpy="0 0 0"/>
-      <geometry>
-    <box size="0.1 0.1 0.1"/>
-      </geometry>
-      <material name="red"/>
-    </visual>
-    <inertial>
-      <mass value="1e-5" />
-      <origin xyz="0 0 0" rpy="0 0 0"/>
-      <inertia ixx="1e-6" ixy="0" ixz="0" iyy="1e-6" iyz="0" izz="1e-6" />
-    </inertial>
-  </link>
-  <!-- Lidar Stand -->
-  <link name="lidar_stand">
+  <link name="castor_cylinder2">
     <visual>
       <geometry>
-        <box size="0.1 0.1 0.75"/>
+        <cylinder length="0.03" radius="0.05"/>
       </geometry>
       <origin rpy="0 0 0" xyz="0 0 0"/>
@@ -210,423 +119,54 @@
     <collision>
       <geometry>
-        <box size="0.1 0.1 0.2"/>
+        <cylinder length="0.03" radius="0.05"/>
       </geometry>
-      <origin rpy="0 0 0" xyz="0 0 0"/>
+      <origin rpy ="0 0 0" xyz="0 0 0"/>
     </collision>
     <inertial>
-      <mass value="0.05"/>
-      <origin rpy="0 0 0" xyz="0 0 0"/>
-      <inertia ixx="0.001" ixy="0" ixz="0" iyy="0.001" iyz="0" izz="0.001"/>
+      <mass value="2"/>
+      <inertia ixx="0.166667" ixy="0.0" ixz="0.0" iyy="0.166667" iyz="0.0" izz="0.166667"/>
     </inertial>
   </link>
-  <!-- IMU Link -->
-  <link name="imu_link">
-    <visual>
-      <geometry>
-        <box size="0.1 0.1 0.1"/>
-      </geometry>
-    </visual>
-    <collision>
-      <geometry>
-        <box size="0.1 0.1 0.1"/>
-      </geometry>
-    </collision>
-    <inertial>
-      <mass value="0.01"/>
-      <inertia ixx="0.001" ixy="0" ixz="0" iyy="0.001" iyz="0" izz="0.001"/>
-    </inertial>
-  </link>
-  <link name = "camera_forward_frame">
-  </link>
-  <joint name = "camera_forward_frame_joint" type="fixed">
+  <!-- JOINTS -->
+  <joint name="footprint_to_baselink" type="fixed">
+    <parent link="base_footprint"/>
+    <child link="base_link"/>
+    <origin rpy ="0 0 0" xyz="0 0 0.13"/>
+  </joint>
+  <joint name="body_to_wheel1" type="continuous">
     <parent link="base_link"/>
-    <child link = "camera_forward_frame"/>
-    <origin xyz="0.2 0 0" rpy="0 0 0"/>
+    <child link="wheel1"/>
+    <axis xyz="-1 0 0"/>
+    <origin rpy ="0 0 1.5707" xyz="0.0 0.28 0"/>
   </joint>
-  <link name = "camera_backward_frame">
-  </link>
-  <joint name = "camera_backward_frame_joint" type="fixed">
+  <joint name="body_to_wheel2" type="continuous">
     <parent link="base_link"/>
-    <child link = "camera_backward_frame"/>
-    <origin xyz="-0.2 0 0" rpy="0 0 3.14"/>
+    <child link="wheel2"/>
+    <axis xyz="1 0 0"/>
+    <origin rpy ="0 0 -1.5707" xyz="0 -0.28 0"/>
   </joint>
-  <link name = "camera_left_frame">
-  </link>
-  <joint name = "camera_left_frame_joint" type="fixed">
+  <joint name="body_to_castor_cylinder" type="continuous">
     <parent link="base_link"/>
-    <child link = "camera_left_frame"/>
-    <origin xyz="0.2 0 0" rpy="0 0 1.57"/>
+    <child link="castor_cylinder"/>
+    <axis xyz="0 0 1"/>
+    <origin rpy ="0 0 0" xyz="-0.50 0 0"/>
   </joint>
-  <link name = "camera_right_frame">
-  </link>
-  <joint name = "camera_right_frame_joint" type="fixed">
+  <joint name="cylinder_to_castor_ball" type="continuous">
+    <parent link="castor_cylinder"/>
+    <child link="castor_ball"/>
+    <axis xyz="0 1 0"/>
+    <origin rpy ="0 0.132544 0" xyz="0 0 -0.065"/>
+  </joint>
+  <joint name="body_to_castor_cylinder2" type="continuous">
     <parent link="base_link"/>
-    <child link = "camera_right_frame"/>
-    <origin xyz="0.2 0 0" rpy="0 0 -1.57"/>
+    <child link="castor_cylinder2"/>
+    <axis xyz="0 0 1"/>
+    <origin rpy ="0 0 0" xyz="0.40 0 0"/>
   </joint>
-  <!-- Joint Between Base Link and Left Wheel -->
-  <joint name="left_wheel_joint" type="continuous">
-    <parent link="base_link"/>
-    <child link="left_wheel"/>
-    <origin xyz="-0.2 0 0" rpy="0 0 0"/>
+  <joint name="cylinder_to_castor_ball2" type="continuous">
+    <parent link="castor_cylinder2"/>
+    <child link="castor_ball2"/>
     <axis xyz="0 1 0"/>
+    <origin rpy ="0 0.132544 0" xyz="0 0 -0.065"/>
   </joint>
-  <joint name="base_footprint_joint" type="fixed">
-    <parent link="base_link"/>
-    <child link="base_footprint"/>
-    <origin rpy="0 0 0" xyz="0 0 0"/>
-  </joint>
-  <!-- Joint Between Base Link and Right Wheel -->
-  <joint name="right_wheel_joint" type="continuous">
-    <parent link="base_link"/>
-    <child link="right_wheel"/>
-    <origin xyz="-0.2 0 0" rpy="0 0 0"/>
-    <axis xyz="0 1 0"/>
-  </joint>
-  <joint name="castor_joint" type="fixed">
-    <parent link="base_link"/>
-    <child link="castor_wheel"/>
-    <origin rpy="0 0 0" xyz="0.35 0 -0.05"/>
-  </joint>
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